Commit message: update foot collision

File: resources/robots/h1_2/h1_2_simplified.urdf (robot description, URDF)
Before this commit: robot h1_5, 56 links, 55 joints
Links:
- link left_ankle_roll_link: geometry collision cylinder length=0.042 radius=0.005; collision cylinder length=0.076 radius=0.005
- link right_ankle_roll_link: geometry collision cylinder length=0.042 radius=0.005; collision cylinder length=0.076 radius=0.005
