Commit message: fix arm joint's range

File: resources/robots/h1_2/h1_2.urdf (robot description, URDF)
Before this commit: robot h1_5, 56 links, 55 joints
Joints:
- joint left_elbow_pitch_joint: limit lower=-2.53 upper=1.6 effort=18 velocity=20 -> lower=-0.95 upper=3.18 effort=18 velocity=20
- joint left_elbow_roll_joint: limit lower=-2.967 upper=2.967 effort=19 velocity=31.4 -> lower=-3.01 upper=2.75 effort=19 velocity=31.4
- joint left_shoulder_yaw_joint: limit lower=-3.01 upper=2.66 effort=18 velocity=20 -> lower=-2.66 upper=3.01 effort=18 velocity=20
- joint left_wrist_pitch_joint: limit lower=-0.471 upper=0.349 effort=19 velocity=31.4 -> lower=-0.47 upper=0.47 effort=19 velocity=31.4
- joint left_wrist_yaw_joint: limit lower=-1.012 upper=1.012 effort=19 velocity=31.4 -> lower=-1.27 upper=1.27 effort=19 velocity=31.4
- joint right_elbow_pitch_joint: limit lower=-1.6 upper=2.53 effort=18 velocity=20 -> lower=-0.95 upper=3.18 effort=18 velocity=20
- joint right_elbow_roll_joint: limit lower=-2.967 upper=2.967 effort=19 velocity=31.4 -> lower=-2.75 upper=3.01 effort=19 velocity=31.4
- joint right_shoulder_pitch_joint: limit lower=-1.57 upper=3.14 effort=40 velocity=9 -> lower=-3.14 upper=1.57 effort=40 velocity=9
- joint right_shoulder_yaw_joint: limit lower=-2.66 upper=3.01 effort=18 velocity=20 -> lower=-3.01 upper=2.66 effort=18 velocity=20
- joint right_wrist_pitch_joint: limit lower=-0.471 upper=0.349 effort=19 velocity=31.4 -> lower=-0.47 upper=0.47 effort=19 velocity=31.4
- joint right_wrist_yaw_joint: limit lower=-1.012 upper=1.012 effort=19 velocity=31.4 -> lower=-1.27 upper=1.27 effort=19 velocity=31.4

File: resources/robots/h1_2/h1_2_simplified.urdf (robot description, URDF)
Before this commit: robot h1_5, 56 links, 55 joints
Joints:
- joint left_elbow_pitch_joint: limit lower=-2.53 upper=1.6 effort=18 velocity=20 -> lower=-0.95 upper=3.18 effort=18 velocity=20
- joint left_elbow_roll_joint: limit lower=-2.967 upper=2.967 effort=19 velocity=31.4 -> lower=-3.01 upper=2.75 effort=19 velocity=31.4
- joint left_shoulder_yaw_joint: limit lower=-3.01 upper=2.66 effort=18 velocity=20 -> lower=-2.66 upper=3.01 effort=18 velocity=20
- joint left_wrist_pitch_joint: limit lower=-0.471 upper=0.349 effort=19 velocity=31.4 -> lower=-0.47 upper=0.47 effort=19 velocity=31.4
- joint left_wrist_yaw_joint: limit lower=-1.012 upper=1.012 effort=19 velocity=31.4 -> lower=-1.27 upper=1.27 effort=19 velocity=31.4
- joint right_elbow_pitch_joint: limit lower=-1.6 upper=2.53 effort=18 velocity=20 -> lower=-0.95 upper=3.18 effort=18 velocity=20
- joint right_elbow_roll_joint: limit lower=-2.967 upper=2.967 effort=19 velocity=31.4 -> lower=-2.75 upper=3.01 effort=19 velocity=31.4
- joint right_shoulder_pitch_joint: limit lower=-1.57 upper=3.14 effort=40 velocity=9 -> lower=-3.14 upper=1.57 effort=40 velocity=9
- joint right_shoulder_yaw_joint: limit lower=-2.66 upper=3.01 effort=18 velocity=20 -> lower=-3.01 upper=2.66 effort=18 velocity=20
- joint right_wrist_pitch_joint: limit lower=-0.471 upper=0.349 effort=19 velocity=31.4 -> lower=-0.47 upper=0.47 effort=19 velocity=31.4
- joint right_wrist_yaw_joint: limit lower=-1.012 upper=1.012 effort=19 velocity=31.4 -> lower=-1.27 upper=1.27 effort=19 velocity=31.4
