Commit message: add h1

File: resources/robots/h1/urdf/h1.urdf (robot description, URDF)
Before this commit: robot h1_description, 22 links, 21 joints
Joints:
- joint left_elbow_joint: type revolute -> fixed
- joint left_shoulder_pitch_joint: type revolute -> fixed
- joint left_shoulder_roll_joint: type revolute -> fixed
- joint left_shoulder_yaw_joint: type revolute -> fixed
- joint right_elbow_joint: type revolute -> fixed
- joint right_shoulder_pitch_joint: type revolute -> fixed
- joint right_shoulder_roll_joint: type revolute -> fixed
- joint right_shoulder_yaw_joint: type revolute -> fixed
- joint torso_joint: type revolute -> fixed

Commit message: update the trainning of g1,h1,h1_2

File: resources/robots/h1/urdf/h1.urdf (robot description, URDF)
Before this commit: robot h1_description, 22 links, 21 joints
Links:
- link left_hip_yaw_link: geometry visual mesh filename=../meshes/left_hip_yaw_link.STL
- link right_hip_yaw_link: geometry visual mesh filename=../meshes/right_hip_yaw_link.STL
