Commit message: Modified g1 urdf with rubber hand and correct collision mesh; Modified deploy_mujoco, deploy_real, and play by using the action of all 29 joint of the g1; Implemented the joint transform to deal with different joint order between the IsaacLab and the low-level controller

File: resources/robots/g1_description/g1_29dof_rev_1_0.urdf (robot description, URDF)
Before this commit: robot g1_29dof_rev_1_0, 39 links, 38 joints
Links:
- link left_ankle_roll_link: geometry collision box size=0.20820672 0.07558269 0.02; visual mesh filename=meshes/left_ankle_roll_link.STL
- link left_rubber_hand: geometry collision box size=0.12 0.03 0.08; visual mesh filename=meshes/left_rubber_hand.STL
- link right_ankle_roll_link: geometry collision box size=0.20820672 0.07558269 0.02; visual mesh filename=meshes/right_ankle_roll_link.STL
- link right_rubber_hand: geometry collision box size=0.12 0.03 0.08; visual mesh filename=meshes/right_rubber_hand.STL
